File: BluePill-SmartNode-RS485.kicad_pcb (KiCad board)
At the start: 4 copper layers, 100 x 80 mm, 32 parts, among them K1 SRD-05VDC, K2 SRD-05VDC, U1 Bluepill_L, U2 Bluepill_R

Commit message: auto-backup 2026-07-18 16:57:53
Routing:
- net 3V3: track 0.00 -> 120.3 mm, vias 0 -> 1
- net PB0: track 0.00 -> 77.8 mm, vias 0 -> 1
- net K2_DRV: track 0.00 -> 74.3 mm
- net K1_DRV: track 0.00 -> 53.0 mm
- net PA2: track 0.00 -> 52.3 mm
- net PA4: track 0.00 -> 47.6 mm
- net PA3: track 0.00 -> 44.1 mm
- net REL1_NC: track 0.00 -> 40.9 mm
- net REL1_NO: track 0.00 -> 37.9 mm
- net REL1_COM: track 0.00 -> 37.2 mm
- net 12V_IN: track 0.00 -> 36.3 mm
- net PA1: track 0.00 -> 36.3 mm
- net PA0: track 0.00 -> 36.3 mm
- net REL2_NC: track 0.00 -> 35.4 mm, vias 0 -> 1
- net PB6: track 0.00 -> 34.5 mm, vias 0 -> 1
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
Commit message: auto-backup 2026-07-19 21:26:17
Parts:
- moved R1 8.85 mm to (78.0, 3.50), turned to 0 degrees
- moved J_REL1 2.10 mm to (71.0, 74.1)
- moved MH2 1.40 mm to (95.0, 3.60)
- moved R_PULL1 0.60 mm to (49.4, 60.0)
Routing:
- net 3V3: track 120.3 -> 161.2 mm
- net LED1_A: track 0.00 -> 8.66 mm
- net REL1_NO: track 37.9 -> 41.6 mm
- net REL1_COM: track 37.2 -> 39.0 mm
- net REL1_NC: track 40.9 -> 42.8 mm
Changed lines of the file:
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@@
 	(footprint "MountingHole:MountingHole_3.2mm"
 		(layer "F.Cu")
-		(at 95 5)
+		(at 95 3.6)
 		(property "Reference" "MH2"
 			(at 0 0 0)
@@
 	(footprint "Resistor_THT:R_Axial_DIN0207_L6.3mm_D2.5mm_P10.16mm_Horizontal"
 		(layer "F.Cu")
-		(at 50 60)
+		(at 49.4 60)
 		(descr "Resistor, Axial_DIN0207 series, Axial, Horizontal, pin pitch=10.16mm, 0.25W = 1/4W, length*diameter=6.3*2.5mm^2, http://cdn-reichelt.de/documents/datenblatt/B400/1_4W%23YAG.pdf")
 		(tags "Resistor Axial_DIN0207 series Axial Horizontal pin pitch 10.16mm 0.25W = 1/4W length 6.3mm diameter 2.5mm")
@@
 	(footprint "Resistor_THT:R_Axial_DIN0207_L6.3mm_D2.5mm_P10.16mm_Horizontal"
 		(layer "F.Cu")
-		(at 84 10 90)
+		(at 78 3.5)
 		(descr "Resistor, Axial_DIN0207 series, Axial, Horizontal, pin pitch=10.16mm, 0.25W = 1/4W, length*diameter=6.3*2.5mm^2, http://cdn-reichelt.de/documents/datenblatt/B400/1_4W%23YAG.pdf")
 		(tags "Resistor Axial_DIN0207 series Axial Horizontal pin pitch 10.16mm 0.25W = 1/4W length 6.3mm diameter 2.5mm")
 		(property "Reference" "R1"
-			(at 5.08 -2.37 90)
+			(at 5.08 -2.37 0)
 			(layer "F.SilkS")
 			(effects
@@
 		)
 		(property "Value" "330R"
-			(at 5.08 2.37 90)
+			(at 5.08 2.37 0)
 			(layer "F.Fab")
 			(effects
@@
 		)
 		(property "Datasheet" ""
-			(at 0 0 90)
+			(at 0 0 0)
 			(layer "F.Fab")
 			(hide yes)
@@
 		)
 		(property "Description" ""
-			(at 0 0 90)
+			(at 0 0 0)
 			(layer "F.Fab")
 			(hide yes)
@@
 		)
 		(property "KiLib_Generator" "resistor/THT"
-			(at 0 0 90)
+			(at 0 0 0)
 			(layer "F.SilkS")
 			(hide yes)
@@
 		(duplicate_pad_numbers_are_jumpers no)
 		(fp_line
+			(start 1.04 0)
+			(end 1.81 0)
+			(stroke
+				(width 0.12)
+				(type solid)
+			)
+			(layer "F.SilkS")
+		)
+		(fp_line
 			(start 9.12 0)
 			(end 8.35 0)
-			(stroke
-				(width 0.12)
-				(type solid)
-			)
-			(layer "F.SilkS")
-		)
-		(fp_line
-			(start 1.04 0)
-			(end 1.81 0)
 			(stroke
 				(width 0.12)
@@
 		)
 		(fp_line
+			(start 0 0)
+			(end 1.93 0)
+			(stroke
+				(width 0.1)
+				(type solid)
+			)
+			(layer "F.Fab")
+		)
+		(fp_line
 			(start 10.16 0)
 			(end 8.23 0)
-			(stroke
-				(width 0.1)
-				(type solid)
-			)
-			(layer "F.Fab")
-		)
-		(fp_line
-			(start 0 0)
-			(end 1.93 0)
 			(stroke
 				(width 0.1)
@@
 		)
 		(fp_text user "${REFERENCE}"
-			(at 5.08 0 90)
+			(at 5.08 0 0)
 			(layer "F.Fab")
 			(effects
@@
 		)
 		(pad "1" thru_hole circle
-			(at 0 0 90)
+			(at 0 0)
 			(size 1.6 1.6)
 			(drill 0.8)
@@
 		)
 		(pad "2" thru_hole circle
-			(at 10.16 0 90)
+			(at 10.16 0)
 			(size 1.6 1.6)
 			(drill 0.8)
@@
 	(footprint "TerminalBlock_Phoenix:TerminalBlock_Phoenix_MKDS-1,5-3-5.08_1x03_P5.08mm_Horizontal"
 		(layer "F.Cu")
-		(at 71 72)
+		(at 71 74.1)
 		(descr "Terminal Block Phoenix MKDS-1,5-3-5.08, 3 pins, pitch 5.08mm, size 15.2x9.8mm, drill diameter 1.3mm, pad diameter 2.6mm, http://www.farnell.com/datasheets/100425.pdf")
 		(tags "THT Terminal Block Phoenix MKDS-1,5-3-5.08 pitch 5.08mm size 15.2x9.8mm drill 1.3mm pad 2.6mm")
@@
 	)
 	(segment
+		(start 62.86 19.08)
+		(end 69.22 25.44)
+		(width 0.4)
+		(layer "B.Cu")
+		(net "3V3")
+	)
+	(segment
+		(start 69.22 25.44)
+		(end 73.36 25.44)
+		(width 0.4)
+		(layer "B.Cu")
+		(net "3V3")
+	)
+	(segment
 		(start 47.18 57.18)
 		(end 50 60)
@@
 		(start 20.525 50.8518)
 		(end 12.8575 58.5193)
+		(width 0.4)
+		(layer "B.Cu")
+		(net "3V3")
+	)
+	(segment
+		(start 73.36 25.44)
+		(end 93 45.08)
 		(width 0.4)
 		(layer "B.Cu")
@@
 	)
 	(segment
-		(start 70.2304 71.2304)
-		(end 71 72)
+		(start 71 74.1)
+		(end 70.2304 71.2304)
 		(width 0.4)
 		(layer "F.Cu")
@@
 	)
 	(segment
-		(start 80.386 71.226)
-		(end 81.16 72)
+		(start 81.16 74.1)
+		(end 80.386 71.226)
 		(width 0.4)
 		(layer "F.Cu")
@@
 	)
 	(segment
-		(start 81.9223 73.8097)
-		(end 83.0129 72.7191)
+		(start 76.08 74.1)
+		(end 83.0129 77)
 		(width 0.4)
 		(layer "F.Cu")
@@
 	)
 	(segment
-		(start 76.08 72)
-		(end 77.8897 73.8097)
-		(width 0.4)
-		(layer "F.Cu")
-		(net "REL1_NO")
-	)
-	(segment
 		(start 81.0877 65.3649)
 		(end 81.0877 48.1123)
@@
 	)
 	(segment
-		(start 77.8897 73.8097)
-		(end 81.9223 73.8097)
+		(start 83.0129 77)
+		(end 83.0129 72.7191)
 		(width 0.4)
 		(layer "F.Cu")
@@
 	)
 	(segment
+		(start 88.16 3.5)
+		(end 89.04 3.5)
+		(width 0.25)
+		(layer "F.Cu")
+		(net "LED1_A")
+	)
+	(segment
+		(start 89.04 3.5)
+		(end 94.54 9)
+		(width 0.25)
+		(layer "F.Cu")
+		(net "LED1_A")
+	)
+	(segment

Commit message: auto-backup 2026-07-20 13:26:17
Routing:
- net 12V_IN: track 36.3 -> 46.3 mm
Changed lines of the file:
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@@
+	)
+	(segment
+		(start 8 27)
+		(end 8 37)
+		(width 0.4)
+		(layer "B.Cu")
+		(net "12V_IN")
 	)
 	(segment
